Commit message: Fixed wheel_separation

File: description/gazebo_control.xacro (robot description, xacro)
@@ -6,10 +6,11 @@
     		<left_joint>left_wheel_joint</left_joint>
     		<right_joint>right_wheel_joint</right_joint>
-    		<wheel_separation>0.28</wheel_separation>
+    		<wheel_separation>0.34</wheel_separation>
+            <!-- 0.31 -->
 			<wheel_radius>0.04</wheel_radius>
             <!-- 0.04 -->
     		<!-- Limits -->
-    		<!-- <max_wheel_torque>200</max_wheel_torque> -->
-            <!-- <max_linear_acceleration>1.0</max_linear_acceleration> -->
+    		<max_wheel_torque>200</max_wheel_torque>
+            <max_linear_acceleration>1.0</max_linear_acceleration>
 			<!-- Input -->
             <topic>cmd_vel</topic>

File: description/lidar.xacro (robot description, xacro)
@@ -26,5 +26,4 @@
 		<material>Gazebo/Red</material>
         <sensor name="laser" type="gpu_lidar">
-            <!-- <ignition_frame_id>custom_name_here</ignition_frame_id>             <pose> 0 0 0 0 0 0 </pose> -->
             <visualize>false</visualize>
             <update_rate>10</update_rate>
@@ -39,5 +38,5 @@
                 <range>
                     <min>0.1</min>
-                    <max>8</max>
+                    <max>12</max>
                 </range>
             </lidar>

File: description/robot_core.xacro (robot description, xacro)
@@ -63,9 +63,16 @@
 	</gazebo>
 	<!-- LEFT WHEEL LINK -->
-	<joint name="left_wheel_joint" type="continuous">
+	<!-- <joint name="left_wheel_joint" type="continuous">
 		<parent link="chassis"/>
 		<child link="left_wheel"/>
 		<origin xyz="0 0.155 0" rpy="-${pi/2} 0 0"/>
 		<axis xyz="0 0 1"/>
+	</joint> -->
+	<joint name="left_wheel_joint" type="continuous">
+		<parent link="chassis"/>
+		<child link="left_wheel"/>
+		<origin xyz="0 0.155 0" rpy="-${pi/2} 0 0"/>
+		<axis xyz="0 0 1"/>
+		<dynamics damping="0.1" friction="0.1"/>
 	</joint>
 	<link name="left_wheel">
@@ -86,13 +93,29 @@
 		</xacro:inertial_cylinder>
 	</link>
+	<!-- <gazebo reference="left_wheel">
+		<material>Gazebo/Blue</material>
+	</gazebo> -->
 	<gazebo reference="left_wheel">
 		<material>Gazebo/Blue</material>
+		<mu1 value="1.0"/>
+		<mu2 value="1.0"/>
+		<kp value="1000000.0"/>
+		<kd value="100.0"/>
+		<minDepth value="0.001"/>
+		<maxVel value="1.0"/>
 	</gazebo>
 	<!-- RIGHT WHEEL LINK -->
-	<joint name="right_wheel_joint" type="continuous">
+	<!-- <joint name="right_wheel_joint" type="continuous">
 		<parent link="chassis"/>
 		<child link="right_wheel"/>
 		<origin xyz="0 -0.155 0" rpy="${pi/2} 0 0"/>
 		<axis xyz="0 0 -1"/>
+	</joint> -->
+	<joint name="right_wheel_joint" type="continuous">
+		<parent link="chassis"/>
+		<child link="right_wheel"/>
+		<origin xyz="0 -0.155 0" rpy="${pi/2} 0 0"/>
+		<axis xyz="0 0 -1"/>
+		<dynamics damping="0.1" friction="0.1"/>
 	</joint>
 	<link name="right_wheel">
@@ -113,6 +136,15 @@
 		</xacro:inertial_cylinder>
 	</link>
+	<!-- <gazebo reference="right_wheel">
+		<material>Gazebo/Blue</material>
+	</gazebo> -->
 	<gazebo reference="right_wheel">
 		<material>Gazebo/Blue</material>
+		<mu1 value="1.0"/>
+		<mu2 value="1.0"/>
+		<kp value="1000000.0"/>
+		<kd value="100.0"/>
+		<minDepth value="0.001"/>
+		<maxVel value="1.0"/>
 	</gazebo>
 	<!-- CASTER WHEEL LINK BACK -->
@@ -141,6 +173,6 @@
 	<gazebo reference="caster_wheel_back">
 		<material>Gazebo/Black</material>
-		<mu1 value="0.001"/>
-		<mu2 value="0.001"/>
+		<mu1 value="0.1"/>
+		<mu2 value="0.1"/>
 	</gazebo>
 	<!-- CASTER WHEEL LINK 2 -->
@@ -169,6 +201,6 @@
 	<gazebo reference="caster_wheel_front">
 		<material>Gazebo/Black</material>
-		<mu1 value="0.001"/>
-		<mu2 value="0.001"/>
+		<mu1 value="0.1"/>
+		<mu2 value="0.1"/>
 	</gazebo>
 </robot>
