Commit message: Add selectable Kobuki robot model
Port the Kobuki TurtleBot 2 base from the sim_kobuki package and make the
robot model selectable with a `robot_model` argument (sim_bot | kobuki) on
rsp.launch.py, launch_sim.launch.py and sim_with_obstacles.launch.py.

The Livox Mid360 of the original model is dropped: it needs the RGL server
plugin and publishes PointCloud2, while everything here consumes a LaserScan
on `scan`. Instead lidar.xacro becomes a `lidar_2d` macro parametrised by
mount point, and the Kobuki carries it above the top plate — the hexagon
standoffs are visual-only geometry, which a gpu_lidar still sees.

Wheel joints allow 40 rad/s instead of the stock 20. Driving at 1.0 m/s while
turning at 2.0 rad/s needs (1.0 + 2.0 * 0.115) / 0.035 = 35 rad/s on the outer
wheel; at 20 rad/s both wheels saturate to the same speed, so the robot loses
steering authority entirely and drives straight at 0.70 m/s.

The generated URDF of the existing model is unchanged, and circumnavigation
holds the same distance with either model (rho_0 = 2.0 m, rms error 0.028 m
for the Kobuki against 0.037 m for the original).

Co-Authored-By: Claude <noreply@anthropic.com>

File: description/lidar.xacro (robot description, xacro)
@@ -1,47 +1,51 @@
 <?xml version="1.0"?>
 <robot xmlns:xacro="http://www.ros.org/wiki/xacro">
-	<joint name="lidar_joint" type="fixed">
-		<parent link="chassis"/>
-		<child link="lidar_frame"/>
-		<origin xyz="0 0 0.1" rpy="0 0 0"/>
-	</joint>
-	<link name="lidar_frame">
-		<visual>
-			<geometry>
-				<cylinder radius="0.03" length="0.04"/>
-			</geometry>
-			<material name="red"/>
-		</visual>
-		<collision>
-			<geometry>
-				<cylinder radius="0.03" length="0.04"/>
-			</geometry>
-			<material name="red"/>
-		</collision>
-		<xacro:inertial_cylinder mass="0.1" radius="0.03" length="0.04">
-			<origin xyz="0 0 0" rpy="0 0 0"/>
-		</xacro:inertial_cylinder>
-	</link>
-	<gazebo reference="lidar_frame">
-		<material>Gazebo/Red</material>
-        <sensor name="laser" type="gpu_lidar">
-            <visualize>false</visualize>
-            <update_rate>10</update_rate>
-            <lidar>
-                <scan>
-                    <horizontal>
-                        <samples>360</samples>
-                        <min_angle>-3.14</min_angle>
-                        <max_angle>3.14</max_angle>
-                    </horizontal>
-                </scan>
-                <range>
-                    <min>0.1</min>
-                    <max>12</max>
-                </range>
-            </lidar>
-            <topic>scan</topic>
-            <gz_frame_id>lidar_frame</gz_frame_id>
-        </sensor>
-    </gazebo>
+	<!-- 2D GPU lidar. Parametrised by mount point so different robot models can
+	     reuse it: reactive_circumnav expects 360 rays over 12 m on `scan`. -->
+	<xacro:macro name="lidar_2d" params="parent:=chassis xyz:='0 0 0.1' samples:=360 range_max:=12">
+		<joint name="lidar_joint" type="fixed">
+			<parent link="${parent}"/>
+			<child link="lidar_frame"/>
+			<origin xyz="${xyz}" rpy="0 0 0"/>
+		</joint>
+		<link name="lidar_frame">
+			<visual>
+				<geometry>
+					<cylinder radius="0.03" length="0.04"/>
+				</geometry>
+				<material name="red"/>
+			</visual>
+			<collision>
+				<geometry>
+					<cylinder radius="0.03" length="0.04"/>
+				</geometry>
+				<material name="red"/>
+			</collision>
+			<xacro:inertial_cylinder mass="0.1" radius="0.03" length="0.04">
+				<origin xyz="0 0 0" rpy="0 0 0"/>
+			</xacro:inertial_cylinder>
+		</link>
+		<gazebo reference="lidar_frame">
+			<material>Gazebo/Red</material>
+			<sensor name="laser" type="gpu_lidar">
+				<visualize>false</visualize>
+				<update_rate>10</update_rate>
+				<lidar>
+					<scan>
+						<horizontal>
+							<samples>${samples}</samples>
+							<min_angle>-3.14</min_angle>
+							<max_angle>3.14</max_angle>
+						</horizontal>
+					</scan>
+					<range>
+						<min>0.1</min>
+						<max>${range_max}</max>
+					</range>
+				</lidar>
+				<topic>scan</topic>
+				<gz_frame_id>lidar_frame</gz_frame_id>
+			</sensor>
+		</gazebo>
+	</xacro:macro>
 </robot>

File: description/robot.urdf.xacro (robot description, xacro)
@@ -5,4 +5,5 @@
     <!-- <xacro:include filename="ros2_control.xacro"/>   Uncommit for ros2_control -->
     <xacro:include filename="lidar.xacro"/>
+    <xacro:lidar_2d parent="chassis" xyz="0 0 0.1"/>
     <!-- <xacro:include filename="tof_sensors.xacro"/> -->
     <xacro:include filename="camera.xacro"/>
